File: pcb_rev1/pcb.kicad_sch (KiCad schematic)
At the start: 88 parts, among them J1 USB_C_Receptacle_USB2.0, J2 TC2030, Q1 NMOS, Q2 NMOS, Q3 PMOS, SW1 SW_Push, U1 BQ297xy, U5 USBLC6-2P6, U6 STM32WB55CGUx, Y1 32k768, Y2 32M

Commit message: revision work
Parts:
- removed C10, C39: 1u, symbol Device:C_Small
- removed C13, C15, C18, C19, C20, C21: 10u, symbol Device:C_Small
- removed C14: 56p, symbol Device:C_Small
- removed C7, C8: 4u7, symbol Device:C_Small
- removed L2: 1u, symbol Device:L
- removed Q3: PMOS, symbol Simulation_SPICE:PMOS
- removed R20: ??, symbol Device:R_Small
- removed RV1: 235-400k, symbol Device:R_Potentiometer_Small
- removed U4: ~, symbol symbol_library:RT6158H
- removed U8: ~, symbol symbol_library:BQ27441-G1
- added C12, C46, C47: 4u7, symbol Device:C_Small
- added C16, C43, C44: 1u, symbol Device:C_Small
- added C45: 10u, symbol Device:C_Small
- added J3: COIL, symbol Connector:Conn_01x02_Pin
- added Q3, Q5: Q_PMOS_DGS, symbol Device:Q_PMOS_DGS
- added R22: 1M, symbol Device:R_Small
- added R23: 330R, symbol Device:R_Small
- added U10: BQ27441-G1, Package_SON:Texas_VSON-HR-12_2.5x4mm_P0.4mm_ThermalVias, symbol symbol_library:BQ27441-G1
- BT1: value 3.7 -> 1S
- C1: value 0.1u -> 100n
- C2: value 47u -> 1u
- C3: value u01 -> 10n
- C5: value u47 -> 470n
- R10: value ?? -> 10k
- R11: value 100k -> 10k
- R2: value 330 -> 220R
- R3, R4, R8: value 5k1 -> 10k
- R5: value 5k1 -> 100k
- R9: value 1M -> 220R
- TH1: value Thermistor -> 10k NTC
- U3: value ~ -> BQ24160
- U7: value ~ -> SSD1306
- U9: value ~ -> LP38691SDX-3.3
Connections:
- net CRG_INT: now also R5.2, U3.7 (INT); no longer R5.1, U3. (USB)
- net CRG_STAT: now also U3.8 (STAT); no longer U3. (USB)
- net GAUGE_GPO: now also U10.12 (GPOUT)
- net GND: now also C2.1, C5.2, Q1.3 (S), R1.1, R13.2, R15.2, R16.2, R19.1, TH1.2, U3.15 (GND), U3.16 (GND), U3.17 (GND), U3.5 (GND), C12.2, C16.2, C43.2, C44.2, C45.2, C46.1, C47.1, J3.2 (Pin_2), R22.2, U10.3 (VSS); no longer C2.2, C5.1, J1.S1 (SHIELD), Q2.3 (S), R1.2, R11.2, R13.1, R15.1, R16.1, R19.2, TH1.1, U3. (USB)
- net LOAD_EN: no longer R11.1
- net OLED_EN: now also R2.1; no longer R10.1
- net SCL: now also U3.3 (SCL), U10.2 (SCL); no longer U3. (USB)
- net SDA: now also U3.4 (SDA), U10.1 (SDA); no longer U3. (USB)
- net USB_D+: now also U3.2 (D+); no longer U3. (USB)
- net USB_D-: now also U3.1 (D-); no longer U3. (USB)
- net VOP: no longer C11.2, C17.2, C22.2, C23.2, C24.2, C25.2, C28.2, C29.2, C30.2, C6.1, C9.2, R10.2, R3.2, R4.2, R5.2, R8.1, U6.1 (VBAT), U6.20 (VDD), U6.23 (VDDRF), U6.34 (VDDSMPS), U6.35 (VDD), U6.40 (VDDUSB), U6.48 (VDD), U6.8 (VDDA), U7.7 (VDD), U9. (OUT), U9.5 (SNS)
- net at Q1.2 (G): now also U1.2 (Cout); no longer U1.3 (Dout)
- net -BATT: now reaches BT1.2 (-), U1.4 (VSS)
- net -BATT: now also C1.2, Q2.3 (S); no longer C1.1, Q1.3 (S)
- net at R9.2: now also R11.2, Q5.2 (G)
- net at U1.6 (V-): now also R1.2; no longer R1.1
- net VBUS: now reaches C4.2, J1.A4 (VBUS), J1.A9 (VBUS), J1.B4 (VBUS), J1.B9 (VBUS), U5.5 (VBUS)
- net VBUS: now also U3.22 (USB); no longer U3. (USB)
- net +BATT: now reaches BT1.1 (+), R6.1
- net +BATT: now also C5.1, U3.11 (BAT), U3.12 (BAT), C16.1, C43.1, R23.1, U10.5 (VDD), U10.6 (BAT), U10.8 (SRP); no longer C1.2, R2.2
- net VCC: now reaches R6.2
- net VCC: now also C36.1, L1.2, R11.1, U3.13 (SYS), U3.14 (SYS), U9.1 (IN), C45.1, Q5.1 (D), U10.7 (SRN); no longer U3. (USB)
- net at C40.2, U7.5 (VDDB): now also C2.2, U7.7 (VDD), Q3.1 (D)
- net at R12.1: now also R13.1, TH1.1, U3.9 (TS); no longer U3. (USB)
- net at U1.5 (BAT): now also C1.1, R23.2; no longer R2.1
- net at J1.A5 (CC1): now also R16.1; no longer R15.2
- net at Q2.2 (G): now also U1.3 (Dout); no longer U1.2 (Cout)
- net at C3.1, L1.1: now also U3.18 (SW); no longer U3. (USB)
- net at J1.B5 (CC2): now also R15.1; no longer R16.2
- net at C3.2: now also U3.19 (BOOT); no longer U3. (USB)
- net VLOAD renamed COIL_CTRL
- removed net VSYS: C2.1, C36.1, L1.2, U3. (USB), U9.1 (IN)
- new net: C44.1, R12.2, U3.6 (DRV)
- new net: C12.1, J1.S1 (SHIELD), R22.1
- new net: C46.2, U3.20 (PMIDI)
- new net: R19.2, U10.10 (BIN)
- new net: Q3.2 (G), R10.1, R2.2
- new net: J3.1 (Pin_1), Q5.3 (S)
- new net: C47.2, U3.23 (PMIDU)
- new net +3V3: C11.2, C17.2, C22.2, C23.2, C24.2, C25.2, C28.2, C29.2, C30.2, C6.1, C9.2, Q3.3 (S), R10.2, R3.2, R4.2, R5.1, R8.1, U6.1 (VBAT), U6.20 (VDD), U6.23 (VDDRF), U6.34 (VDDSMPS), U6.35 (VDD), U6.40 (VDDUSB), U6.48 (VDD), U6.8 (VDDA), U9. (OUT), U9.5 (SNS)
- no-connect marks 9 -> 10
Other:
- note added: "Power Calculation (P = U²/R, I = U/R): 1.5R @ 4.2V (full) -> 11.76W, 2.8A 1.5R @ 3.7V (empty) -> 9.13W, 2.47A"
- note added: "check if GPIO is 5V tolerant!"
- note added: "seems like you'll be limited to 100mA charge current if not charging with a dedicated charger (PC etc.) You'll probably have to increase it manually via I2C"
- note removed: "FB Voltage Divider Calculator: https://www.desmos.com/calculator/6lxsvs1vco"
- note removed: "General Notes: - Generally 'positive Voltages' point up (Vcc) and 'negative voltages' point down (GND) - Some component values are missing"
- note removed: "I dont think I set up this voltage divider correctly. the idea is to be able to set the output voltage from 2.8-4.2V"
- note removed: "J1: This is a bit controversial, everyone does it a bit different. I usually go for 1MOhm || 4.7nF between shield and GND"
- note removed: "J1: USB-Spec calls for 10uF on VBus"
- note removed: "Note: Using global notes works, but it's more common to use power symbols for this instead (shows the voltage better)"
- note removed: "Pin Numbers missing for U3?"
- note removed: "Probably some more stuff to be fixed, but redrawing would make it easier =)"
- note removed: "SHORT! Bypass with 1uF to PGND"
- note removed: "TS Voltage Divider Calculator: https://www.desmos.com/calculator/g1khjlpplq https://www.lasercalculator.com/ntc-thermistor-calculator"
- note removed: "U8 - BAT: 'connect 1uF to GND'"
- note removed: "U8 - GPOUT: 10k pullup is recommended"
- note removed: "use 10k"
- note removed: "~1.5 Ohm external load"
- moved on the sheet: AE1, BT1, C1, C11, C17, C22, C23, C24, C25, C26, C27, C28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

Commit message: revision work; assign components and MPNs (digikey)
Parts:
- removed D1: LED_RGBA, symbol Device:LED_RGBA
- removed J2: TC2030, Connector:Tag-Connect_TC2030-IDC-FP_2x03_P1.27mm_Vertical, symbol Connector:Conn_ARM_SWD_TagConnect_TC2030
- removed L3, L4: 10n, symbol Device:L_Small
- removed Q1, Q2: NMOS, symbol Simulation_SPICE:NMOS
- removed Q3, Q5: Q_PMOS_DGS, symbol Device:Q_PMOS_DGS
- removed R14: R_Small, symbol Device:R_Small
- removed R21: 5k1, symbol Device:R_Small
- removed U3: BQ24160, symbol symbol_library:BQ24160
- added D1: ~, LED_SMD:MSL0104RGBU1, symbol LED:MSL0104RGBU1
- added J2: TC2030, Connector:Tag-Connect_TC2030-IDC-NL_2x03_P1.27mm_Vertical, symbol Connector_Generic:Conn_01x06
- added L1: 10n, Capacitor_SMD:C_0603_1608Metric, symbol Device:L_Small
- added L2: 10u, Inductor_SMD:L_Abracon_ASPI-3012S, symbol Device:L
- added Q1, Q4: SSM3J338R, Package_TO_SOT_SMD:SOT-23, symbol Device:Q_PMOS_GSD
- added Q2, Q3: DMN3023L-7, Package_TO_SOT_SMD:SOT-23, symbol Device:Q_NMOS_GSD
- added R7, R8, R9: 1k, Resistor_SMD:R_0603_1608Metric, symbol Device:R_Small
- added U7: BQ24160, Package_DFN_QFN:QFN-24-1EP_4x4mm_P0.5mm_EP2.7x2.7mm_ThermalVias, symbol symbol_library:BQ24160
- AE1: footprint (none) -> RF_Antenna:Johanson_2500AT44M0400
- BT1: footprint (none) -> Connector_PinHeader_2.54mm:PinHeader_1x02_P2.54mm_Vertical; now not fitted
- C1: renamed from C24; footprint (none) -> Capacitor_SMD:C_0603_1608Metric; Digikey_MPN (none) -> C0603C104K5RAC7411
- C10: renamed from C25; footprint (none) -> Capacitor_SMD:C_1206_3216Metric; Digikey_MPN (none) -> C1206C475K5RAC7800
- C11: renamed from C34; footprint (none) -> Capacitor_SMD:C_0603_1608Metric; Digikey_MPN (none) -> C0603C104K5RAC7411
- C12: renamed from C31; footprint (none) -> Capacitor_SMD:C_1206_3216Metric; Digikey_MPN (none) -> C1206C475K5RAC7800
- C13: renamed from C27; value 0p8 -> 1p; footprint (none) -> Capacitor_SMD:C_0603_1608Metric; Digikey_MPN (none) -> C0603C109C5GAC7867
- C14: renamed from C26; value 0p3 -> 1p1; footprint (none) -> Capacitor_SMD:C_0603_1608Metric; Digikey_MPN (none) -> CBR06C119B5GAC
- C15: renamed from C35; value ?? -> 100n; footprint (none) -> Capacitor_SMD:C_0603_1608Metric; Digikey_MPN (none) -> C0603C104K5RAC7411
- C16: renamed from C32; value 10p -> 20p; footprint (none) -> Capacitor_SMD:C_0603_1608Metric; Digikey_MPN (none) -> C0603C200K5GAC7867
- C17: renamed from C33; value 10p -> 20p; footprint (none) -> Capacitor_SMD:C_0603_1608Metric; Digikey_MPN (none) -> C0603C200K5GAC7867
- C18: renamed from C5; value 470n -> 1u; footprint (none) -> Capacitor_SMD:C_0805_2012Metric; Digikey_MPN (none) -> C0805C105K5RAC7800
- C19: renamed from C16; footprint (none) -> Capacitor_SMD:C_0805_2012Metric; Digikey_MPN (none) -> C0805C105K5RAC7800
- C2: renamed from C23; footprint (none) -> Capacitor_SMD:C_0603_1608Metric; Digikey_MPN (none) -> C0603C104K5RAC7411
- C20: renamed from C1; footprint (none) -> Capacitor_SMD:C_0603_1608Metric; Digikey_MPN (none) -> C0603C104K5RAC7411
- C21: renamed from C40; footprint (none) -> Capacitor_SMD:C_0805_2012Metric; Digikey_MPN (none) -> C0805C105K5RAC7800
- C22: renamed from C2; footprint (none) -> Capacitor_SMD:C_0805_2012Metric; Digikey_MPN (none) -> C0805C105K5RAC7800
- C23: renamed from C37; footprint (none) -> Capacitor_SMD:C_0805_2012Metric; Digikey_MPN (none) -> C0805C105K5RAC7800
- C24: renamed from C38; footprint (none) -> Capacitor_SMD:C_0805_2012Metric; Digikey_MPN (none) -> C0805C105K5RAC7800
- C25: renamed from C3; footprint (none) -> Capacitor_SMD:C_0603_1608Metric; Digikey_MPN (none) -> C0603C103K5RAC7867
- C26: renamed from C36; footprint (none) -> Capacitor_SMD:C_0805_2012Metric; Digikey_MPN (none) -> C0805C105K5RAC7800
- C27: renamed from C6; footprint (none) -> Capacitor_SMD:C_0805_2012Metric; Digikey_MPN (none) -> C0805C105K5RAC7800
- C28: renamed from C4; footprint (none) -> Capacitor_SMD:C_0805_2012Metric; Digikey_MPN (none) -> C0805C105K5RAC7800
- C29: renamed from C41; footprint (none) -> Capacitor_SMD:C_1206_3216Metric; Digikey_MPN (none) -> C1206C225K5RAC7800
- C3: renamed from C22; footprint (none) -> Capacitor_SMD:C_0603_1608Metric; Digikey_MPN (none) -> C0603C104K5RAC7411
- C30: renamed from C42; footprint (none) -> Capacitor_SMD:C_1206_3216Metric; Digikey_MPN (none) -> C1206C475K5RAC7800
- C31: renamed from C45; footprint (none) -> Capacitor_SMD:C_1206_3216Metric; Digikey_MPN (none) -> C1210C106K5RAC7800
- C32: renamed from C43; footprint (none) -> Capacitor_SMD:C_0805_2012Metric; Digikey_MPN (none) -> C0805C105K5RAC7800
- C33: renamed from C46; footprint (none) -> Capacitor_SMD:C_1206_3216Metric; Digikey_MPN (none) -> C1206C475K5RAC7800
- C34: renamed from C47; footprint (none) -> Capacitor_SMD:C_1206_3216Metric; Digikey_MPN (none) -> C1206C475K5RAC7800
- C35: renamed from C44; footprint (none) -> Capacitor_SMD:C_0805_2012Metric; Digikey_MPN (none) -> C0805C105K5RAC7800
- C36: renamed from C12; footprint (none) -> Capacitor_SMD:C_1206_3216Metric; Digikey_MPN (none) -> C1206C475K5RAC7800
- C4: renamed from C17; footprint (none) -> Capacitor_SMD:C_0603_1608Metric; Digikey_MPN (none) -> C0603C104K5RAC7411
- C5: renamed from C11; footprint (none) -> Capacitor_SMD:C_0603_1608Metric; Digikey_MPN (none) -> C0603C104K5RAC7411
- C6: renamed from C9; footprint (none) -> Capacitor_SMD:C_0603_1608Metric; Digikey_MPN (none) -> C0603C104K5RAC7411
- C7: renamed from C30; footprint (none) -> Capacitor_SMD:C_0603_1608Metric; Digikey_MPN (none) -> C0603C104K5RAC7411
- C8: renamed from C28; footprint (none) -> Capacitor_SMD:C_0603_1608Metric; Digikey_MPN (none) -> C0603C104K5RAC7411
- C9: renamed from C29; footprint (none) -> Capacitor_SMD:C_1206_3216Metric; Digikey_MPN (none) -> C1206C475K5RAC7800
- J1: renamed from J3; footprint (none) -> Connector_PinHeader_2.54mm:PinHeader_1x02_P2.54mm_Vertical
- J3: renamed from J1; footprint (none) -> Connector_USB:USB_C_Receptacle_GCT_USB4105-xx-A_16P_TopMnt_Horizontal; Digikey_MPN (none) -> 2073-USB4105-GF-ATR-ND
- L3: renamed from L5; value 2n2 -> 2n7; footprint (none) -> Capacitor_SMD:C_0603_1608Metric; Digikey_MPN (none) -> 712-LRC0603CS2N7GV001TTR-ND; Distrubuter Link https://www.digikey.com/en/products/detail/murata-electroni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 -> https://www.digikey.com/en/products/detail/johanson-technol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
- L4: renamed from L1; footprint (none) -> Inductor_SMD:L_Abracon_ASPI-3012S; Digikey_MPN (none) -> 535-ASPI-3012S-1R5N-TTR-ND
- R1: renamed from R11; footprint (none) -> Resistor_SMD:R_0603_1608Metric; Digikey_MPN (none) -> RC0603FR-0710KL
- R10: renamed from R8; footprint (none) -> Resistor_SMD:R_0603_1608Metric; Digikey_MPN (none) -> RC0603FR-0710KL
- R11: renamed from R6; Digikey_MPN (none) -> RL1206FR-070R01L
- R12: renamed from R23; footprint (none) -> Resistor_SMD:R_0603_1608Metric; Digikey_MPN (none) -> RC0603FR-07330RL
- R13: renamed from R19; footprint (none) -> Resistor_SMD:R_0603_1608Metric; Digikey_MPN (none) -> RC0603FR-0710KL
- R14: renamed from R1; footprint (none) -> Resistor_SMD:R_0603_1608Metric; Digikey_MPN (none) -> RC0603FR-132K2L
- R15: renamed from R2; value 220R -> 330R; footprint (none) -> Resistor_SMD:R_0603_1608Metric; Digikey_MPN (none) -> RC0603FR-07330RL
- R16: renamed from R10; footprint (none) -> Resistor_SMD:R_0603_1608Metric; Digikey_MPN (none) -> RC0603FR-0710KL
- R17: renamed from R7; footprint (none) -> Resistor_SMD:R_0603_1608Metric; Digikey_MPN (none) -> RC0603FR-07390KL
- R18: renamed from R5; footprint (none) -> Resistor_SMD:R_0603_1608Metric; Digikey_MPN (none) -> RC0603FR-07100KL
- R19: renamed from R12; footprint (none) -> Resistor_SMD:R_0603_1608Metric; Digikey_MPN (none) -> RC0603FR-074K7L
- R2: renamed from R9; value 220R -> 330R; footprint (none) -> Resistor_SMD:R_0603_1608Metric; Digikey_MPN (none) -> RC0603FR-07330RL
- R20: renamed from R15; footprint (none) -> Resistor_SMD:R_0603_1608Metric; Digikey_MPN (none) -> RC0603FR-075K1L
- R21: renamed from R16; footprint (none) -> Resistor_SMD:R_0603_1608Metric; Digikey_MPN (none) -> RC0603FR-075K1L
- R22: renamed from R13; value 10k8 -> 10k7; footprint (none) -> Resistor_SMD:R_0603_1608Metric; Digikey_MPN (none) -> RC0603FR-0710K7L
- R23: renamed from R22; footprint (none) -> Resistor_SMD:R_0603_1608Metric; Digikey_MPN (none) -> RC0603FR-071ML
- R3, R4: footprint (none) -> Resistor_SMD:R_0603_1608Metric; Digikey_MPN (none) -> RC0603FR-0710KL
- R5: renamed from R17; value R_Small -> 10k; footprint (none) -> Resistor_SMD:R_0603_1608Metric; Digikey_MPN (none) -> RC0603FR-0710KL
- R6: renamed from R18; value R_Small -> 1k; footprint (none) -> Resistor_SMD:R_0603_1608Metric; Digikey_MPN (none) -> RC0603FR-071KL
- SW1: footprint (none) -> Connector_PinHeader_2.54mm:PinHeader_1x02_P2.54mm_Vertical; Digikey_MPN (none) -> SW1020TR-ND
- TH1: footprint (none) -> TestPoint:TestPoint_Bridge_Pitch2.0mm_Drill0.7mm; Digikey_MPN (none) -> 490-NXFT15XV103FEAB040TR-ND
- U1: renamed from U6; value STM32WB55CGUx -> STM32WB55CGU6; Digikey_MPN (none) -> 497-18489-ND
- U2: value ~ -> DEA102700LT-6307A2; footprint (none) -> Filter:RF_LPF_0402_4Pin; Digikey_MPN (none) -> 445-175598-2-ND
- U3: renamed from U10; value BQ27441-G1 -> BQ27441DRZR-G1A; Digikey_MPN (none) -> 296-39941-2-ND
- U5: renamed from U7; footprint (none) -> Connector_FFC-FPC:FH26W15S03SHW60; Digikey_MPN (none) -> H125791TR-ND; Distrubuter Link https://www.digikey.com/en/products/detail/midas-displays/M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 -> https://www.digikey.com/en/products/detail/hirose-electric-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; MPN_OLED (none) -> 3086-MCOT128032CY-WS-ND
- U6: renamed from U9; footprint (none) -> Package_SON:WSON-6-1EP_3x3mm_P0.95mm; Digikey_MPN (none) -> 296-LP38691SDX-3.3/NOPBTR-ND
- U8: renamed from U5; Digikey_MPN (none) -> 497-5026-2-ND
- Y1: renamed from Y2; footprint (none) -> Crystal:Crystal_SMD_Abracon_ABM8G-4Pin_3.2x2.5mm; Digikey_MPN (none) -> 535-10302-2-ND; Distrubuter Link https://www.digikey.com/en/products/detail/ecliptek/EC3625E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 -> https://www.digikey.com/en/products/detail/abracon-llc/ABM8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
- Y2: renamed from Y1; footprint (none) -> Crystal:Abracon_ABS06_2.0x1.2mm
- renumbered U1 to U4
Connections:
- net VOP is gone; now on net GND: SW1.1
- net +3V3: now also R5.1, U6.4 (OUT), D1.1 (A(R)), D1.2 (A(G)), D1.6 (A(B)), D1.7 (A(R)), J2.1 (Pin_1), Q4.2 (S); no longer U6. (OUT)
- net +BATT: now also U7.11 (BAT), U7.12 (BAT)
- net -BATT: now also Q3.2 (S)
- net CRG_INT: now also U7.7 (INT)
- net CRG_STAT: now also U7.8 (STAT)
- net GND: now also C12.1, C13.2, C14.2, U6.7 (GND), J2.6 (Pin_6), Q2.2 (S), U7.15 (GND), U7.16 (GND), U7.17 (GND), U7.5 (GND); no longer AE1.1 (FEED), C12.2, C13.1, C14.1, R5.2
- net SCL: now also U7.3 (SCL)
- net SDA: now also U7.4 (SDA)
- net STM_RST : now also J2.2 (Pin_2)
- net USB_D+: now also U7.2 (D+)
- net USB_D-: now also U7.1 (D-)
- net VBUS: now also U7.22 (USB)
- net at Y1.1: now also U1.24 (OSC_OUT)
- net at U4.2 (Cout): now also Q2.1 (G)
- net at U1.31 (VFBSMPS): now also C12.2, L2.2; no longer C12.1
- net at U1.33 (VLXSMPS): now also L1.2
- net at U1.39 (PA13): now also J2.4 (Pin_4)
- net at C15.1, R6.2, U1.4 (PH3): now also R5.2; no longer R5.1
- net at U1.41 (PA14): now also J2.3 (Pin_3)
- net at U1.43 (PB3): now also J2.5 (Pin_5)
- net CRG_~{EN}: now reaches U1.44 (PB4)
- net CRG_~{EN}: now also U7.24 (~{DC})
- net at U1.47 (PB7): now also R7.2
- net at U1.5 (PB8): now also R8.2
- net at U1.6 (PB9): now also R9.2
- net at C35.1, R19.2: now also U7.6 (DRV)
- net at C21.2, C22.2, U5.5 (VDDB)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: now also Q4.3 (D)
- net at R1.2, R2.2: now also Q1.1 (G)
- net at C33.2: now also U7.20 (PMIDI)
- net at R19.1, R22.1, TH1.1: now also U7.9 (TS)
- net at R15.2, R16.1: now also Q4.1 (G)
- net at U2.3 (OUT): now also C13.1, L3.2; no longer AE1.2 (PCB_Trace)
- net at U4.3 (Dout): now also Q3.1 (G)
- net at J1.1 (Pin_1): now also Q1.2 (S)
- net at C34.2: now also U7.23 (PMIDU)
- net at C25.1, L4.1: now also U7.18 (SW)
- net at C25.2: now also U7.19 (BOOT)
- net VCC renamed IN
- net IN: now also U6.6 (IN), Q1.3 (D), U7.13 (SYS), U7.14 (SYS)
- new net: AE1.1 (FEED), C14.1, L3.1
- new net: U1.21 (RF1), U2.1 (IN)
- new net: L1.1, L2.1
- new net: D1.3 (K(G)), R8.1
- new net: D1.4 (K(R)), R7.1
- new net: D1.5 (K(B)), R9.1
- new net: Q2.3 (D), Q3.3 (D)
Other:
- note removed: "D1 has two options to work correctly: A: Either R21 goes to Vcc, and the pins sink the current to GND B: D1 is rotated 180° and the pins source current from Vcc Both would work"
- note removed: "OK (just redraw)"
- note removed: "Y2: missing load capacitors (like at Y1)"
- note removed: "why two inductors?"
- moved on the sheet: AE1, C1, C10, C11, C12, C13, C14, C15, C16, C17, C18, C19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
